Commit message: Exercise 8

File: kuka_iiwa_support/urdf/kuka_iiwa.xacro (robot description, xacro)
@@ -1,5 +1,5 @@
 <?xml version="1.0"?>
 <robot name="kuka_iiwa" xmlns:xacro="http://www.ros.org/wiki/xacro">
-  <xacro:include filename="$(find iiwa_description)/urdf/utilities.xacro" />
+  <xacro:include filename="$(find kuka_iiwa_support)/urdf/utilities.xacro" />
   <xacro:include filename="$(find kuka_iiwa_support)/urdf/kuka_iiwa_macro.xacro"/>
   <xacro:arg name="robot_name" default="iiwa"/>

File: kuka_iiwa_support/urdf/kuka_iiwa_ctrl.xacro (robot description, xacro)
@@ -1,5 +1,5 @@
 <?xml version="1.0"?>
 <robot name="kuka_iiwa" xmlns:xacro="http://www.ros.org/wiki/xacro">
-  <xacro:include filename="$(find iiwa_description)/urdf/utilities.xacro" />
+  <xacro:include filename="$(find kuka_iiwa_support)/urdf/utilities.xacro" />
   <xacro:include filename="$(find kuka_iiwa_support)/urdf/kuka_iiwa_macro_ctrl.xacro"/>
   <xacro:arg name="robot_name" default="iiwa"/>

File: kuka_iiwa_support/urdf/kuka_iiwa_macro.xacro (robot description, xacro)
@@ -22,12 +22,12 @@
         <origin xyz="0 0 0" rpy="0 0 0"/>
         <geometry>
-          <mesh filename="package://iiwa_description/meshes/iiwa7/visual/link_0.stl"/>
-        </geometry>
-        <material name="Grey"/>
-      </visual>
-      <collision>
-        <origin xyz="0 0 0" rpy="0 0 0"/>
-        <geometry>
-          <mesh filename="package://iiwa_description/meshes/iiwa7/collision/link_0.stl"/>
+          <mesh filename="package://kuka_iiwa_support/meshes/iiwa7/visual/link_0.stl"/>
+        </geometry>
+        <material name="Grey"/>
+      </visual>
+      <collision>
+        <origin xyz="0 0 0" rpy="0 0 0"/>
+        <geometry>
+          <mesh filename="package://kuka_iiwa_support/meshes/iiwa7/collision/link_0.stl"/>
         </geometry>
         <material name="Grey"/>
@@ -58,5 +58,5 @@
         <origin xyz="0 0 0.0075" rpy="0 0 0"/>
         <geometry>
-          <mesh filename="package://iiwa_description/meshes/iiwa7/visual/link_1.stl"/>
+          <mesh filename="package://kuka_iiwa_support/meshes/iiwa7/visual/link_1.stl"/>
         </geometry>
         <material name="Orange"/>
@@ -65,5 +65,5 @@
         <origin xyz="0 0 0.0075" rpy="0 0 0"/>
         <geometry>
-          <mesh filename="package://iiwa_description/meshes/iiwa7/collision/link_1.stl"/>
+          <mesh filename="package://kuka_iiwa_support/meshes/iiwa7/collision/link_1.stl"/>
         </geometry>
         <material name="Orange"/>
@@ -92,12 +92,12 @@
         <origin xyz="0 0 0" rpy="0 0 0"/>
         <geometry>
-          <mesh filename="package://iiwa_description/meshes/iiwa7/visual/link_2.stl"/>
-        </geometry>
-        <material name="Orange"/>
-      </visual>
-      <collision>
-        <origin xyz="0 0 0" rpy="0 0 0"/>
-        <geometry>
-          <mesh filename="package://iiwa_description/meshes/iiwa7/collision/link_2.stl"/>
+          <mesh filename="package://kuka_iiwa_support/meshes/iiwa7/visual/link_2.stl"/>
+        </geometry>
+        <material name="Orange"/>
+      </visual>
+      <collision>
+        <origin xyz="0 0 0" rpy="0 0 0"/>
+        <geometry>
+          <mesh filename="package://kuka_iiwa_support/meshes/iiwa7/collision/link_2.stl"/>
         </geometry>
         <material name="Orange"/>
@@ -121,12 +121,12 @@
         <origin xyz="0 0 -0.026" rpy="0 0 0"/>
         <geometry>
-          <mesh filename="package://iiwa_description/meshes/iiwa7/visual/link_3.stl"/>
-        </geometry>
-        <material name="Orange"/>
-      </visual>
-      <collision>
-        <origin xyz="0 0 -0.026" rpy="0 0 0"/>
-        <geometry>
-          <mesh filename="package://iiwa_description/meshes/iiwa7/collision/link_3.stl"/>
+          <mesh filename="package://kuka_iiwa_support/meshes/iiwa7/visual/link_3.stl"/>
+        </geometry>
+        <material name="Orange"/>
+      </visual>
+      <collision>
+        <origin xyz="0 0 -0.026" rpy="0 0 0"/>
+        <geometry>
+          <mesh filename="package://kuka_iiwa_support/meshes/iiwa7/collision/link_3.stl"/>
         </geometry>
         <material name="Orange"/>
@@ -150,12 +150,12 @@
         <origin xyz="0 0 0" rpy="0 0 0"/>
         <geometry>
-          <mesh filename="package://iiwa_description/meshes/iiwa7/visual/link_4.stl"/>
-        </geometry>
-        <material name="Orange"/>
-      </visual>
-      <collision>
-        <origin xyz="0 0 0" rpy="0 0 0"/>
-        <geometry>
-          <mesh filename="package://iiwa_description/meshes/iiwa7/collision/link_4.stl"/>
+          <mesh filename="package://kuka_iiwa_support/meshes/iiwa7/visual/link_4.stl"/>
+        </geometry>
+        <material name="Orange"/>
+      </visual>
+      <collision>
+        <origin xyz="0 0 0" rpy="0 0 0"/>
+        <geometry>
+          <mesh filename="package://kuka_iiwa_support/meshes/iiwa7/collision/link_4.stl"/>
         </geometry>
         <material name="Orange"/>
@@ -179,12 +179,12 @@
         <origin xyz="0 0 -0.026" rpy="0 0 0"/>
         <geometry>
-          <mesh filename="package://iiwa_description/meshes/iiwa7/visual/link_5.stl"/>
-        </geometry>
-        <material name="Orange"/>
-      </visual>
-      <collision>
-        <origin xyz="0 0 -0.026" rpy="0 0 0"/>
-        <geometry>
-          <mesh filename="package://iiwa_description/meshes/iiwa7/collision/link_5.stl"/>
+          <mesh filename="package://kuka_iiwa_support/meshes/iiwa7/visual/link_5.stl"/>
+        </geometry>
+        <material name="Orange"/>
+      </visual>
+      <collision>
+        <origin xyz="0 0 -0.026" rpy="0 0 0"/>
+        <geometry>
+          <mesh filename="package://kuka_iiwa_support/meshes/iiwa7/collision/link_5.stl"/>
         </geometry>
         <material name="Orange"/>
@@ -208,12 +208,12 @@
         <origin xyz="0 0 0" rpy="0 0 0"/>
         <geometry>
-          <mesh filename="package://iiwa_description/meshes/iiwa7/visual/link_6.stl"/>
-        </geometry>
-        <material name="Orange"/>
-      </visual>
-      <collision>
-        <origin xyz="0 0 0" rpy="0 0 0"/>
-        <geometry>
-          <mesh filename="package://iiwa_description/meshes/iiwa7/collision/link_6.stl"/>
+          <mesh filename="package://kuka_iiwa_support/meshes/iiwa7/visual/link_6.stl"/>
+        </geometry>
+        <material name="Orange"/>
+      </visual>
+      <collision>
+        <origin xyz="0 0 0" rpy="0 0 0"/>
+        <geometry>
+          <mesh filename="package://kuka_iiwa_support/meshes/iiwa7/collision/link_6.stl"/>
         </geometry>
         <material name="Orange"/>
@@ -237,5 +237,5 @@
         <origin xyz="0 0 -0.0005" rpy="0 0 0"/>
         <geometry>
-          <mesh filename="package://iiwa_description/meshes/iiwa7/visual/link_7.stl"/>
+          <mesh filename="package://kuka_iiwa_support/meshes/iiwa7/visual/link_7.stl"/>
         </geometry>
         <material name="Grey"/>
@@ -244,5 +244,5 @@
         <origin xyz="0 0 -0.0005" rpy="0 0 0"/>
         <geometry>
-          <mesh filename="package://iiwa_description/meshes/iiwa7/collision/link_7.stl"/>
+          <mesh filename="package://kuka_iiwa_support/meshes/iiwa7/collision/link_7.stl"/>
         </geometry>
         <material name="Grey"/>

File: kuka_iiwa_support/urdf/kuka_iiwa_macro_ctrl.xacro (robot description, xacro)
@@ -34,5 +34,5 @@
         <origin xyz="0 0 0" rpy="0 0 0"/>
         <geometry>
-          <mesh filename="package://iiwa_description/meshes/iiwa7/visual/link_0.stl"/>
+          <mesh filename="package://kuka_iiwa_support/meshes/iiwa7/visual/link_0.stl"/>
         </geometry>
         <material name="Grey"/>
@@ -41,5 +41,5 @@
         <origin xyz="0 0 0" rpy="0 0 0"/>
         <geometry>
-          <mesh filename="package://iiwa_description/meshes/iiwa7/collision/link_0.stl"/>
+          <mesh filename="package://kuka_iiwa_support/meshes/iiwa7/collision/link_0.stl"/>
         </geometry>
         <material name="Grey"/>
@@ -70,5 +70,5 @@
         <origin xyz="0 0 0.0075" rpy="0 0 0"/>
         <geometry>
-          <mesh filename="package://iiwa_description/meshes/iiwa7/visual/link_1.stl"/>
+          <mesh filename="package://kuka_iiwa_support/meshes/iiwa7/visual/link_1.stl"/>
         </geometry>
         <material name="Orange"/>
@@ -77,5 +77,5 @@
         <origin xyz="0 0 0.0075" rpy="0 0 0"/>
         <geometry>
-          <mesh filename="package://iiwa_description/meshes/iiwa7/collision/link_1.stl"/>
+          <mesh filename="package://kuka_iiwa_support/meshes/iiwa7/collision/link_1.stl"/>
         </geometry>
         <material name="Orange"/>
@@ -104,12 +104,12 @@
         <origin xyz="0 0 0" rpy="0 0 0"/>
         <geometry>
-          <mesh filename="package://iiwa_description/meshes/iiwa7/visual/link_2.stl"/>
-        </geometry>
-        <material name="Orange"/>
-      </visual>
-      <collision>
-        <origin xyz="0 0 0" rpy="0 0 0"/>
-        <geometry>
-          <mesh filename="package://iiwa_description/meshes/iiwa7/collision/link_2.stl"/>
+          <mesh filename="package://kuka_iiwa_support/meshes/iiwa7/visual/link_2.stl"/>
+        </geometry>
+        <material name="Orange"/>
+      </visual>
+      <collision>
+        <origin xyz="0 0 0" rpy="0 0 0"/>
+        <geometry>
+          <mesh filename="package://kuka_iiwa_support/meshes/iiwa7/collision/link_2.stl"/>
         </geometry>
         <material name="Orange"/>
@@ -133,5 +133,5 @@
         <origin xyz="0 0 -0.026" rpy="0 0 0"/>
         <geometry>
-          <mesh filename="package://iiwa_description/meshes/iiwa7/visual/link_3.stl"/>
+          <mesh filename="package://kuka_iiwa_support/meshes/iiwa7/visual/link_3.stl"/>
         </geometry>
         <material name="Orange"/>
@@ -140,5 +140,5 @@
         <origin xyz="0 0 -0.026" rpy="0 0 0"/>
         <geometry>
-          <mesh filename="package://iiwa_description/meshes/iiwa7/collision/link_3.stl"/>
+          <mesh filename="package://kuka_iiwa_support/meshes/iiwa7/collision/link_3.stl"/>
         </geometry>
         <material name="Orange"/>
@@ -162,12 +162,12 @@
         <origin xyz="0 0 0" rpy="0 0 0"/>
         <geometry>
-          <mesh filename="package://iiwa_description/meshes/iiwa7/visual/link_4.stl"/>
-        </geometry>
-        <material name="Orange"/>
-      </visual>
-      <collision>
-        <origin xyz="0 0 0" rpy="0 0 0"/>
-        <geometry>
-          <mesh filename="package://iiwa_description/meshes/iiwa7/collision/link_4.stl"/>
+          <mesh filename="package://kuka_iiwa_support/meshes/iiwa7/visual/link_4.stl"/>
+        </geometry>
+        <material name="Orange"/>
+      </visual>
+      <collision>
+        <origin xyz="0 0 0" rpy="0 0 0"/>
+        <geometry>
+          <mesh filename="package://kuka_iiwa_support/meshes/iiwa7/collision/link_4.stl"/>
         </geometry>
         <material name="Orange"/>
@@ -191,5 +191,5 @@
         <origin xyz="0 0 -0.026" rpy="0 0 0"/>
         <geometry>
-          <mesh filename="package://iiwa_description/meshes/iiwa7/visual/link_5.stl"/>
+          <mesh filename="package://kuka_iiwa_support/meshes/iiwa7/visual/link_5.stl"/>
         </geometry>
         <material name="Orange"/>
@@ -198,5 +198,5 @@
         <origin xyz="0 0 -0.026" rpy="0 0 0"/>
         <geometry>
-          <mesh filename="package://iiwa_description/meshes/iiwa7/collision/link_5.stl"/>
+          <mesh filename="package://kuka_iiwa_support/meshes/iiwa7/collision/link_5.stl"/>
         </geometry>
         <material name="Orange"/>
@@ -220,12 +220,12 @@
         <origin xyz="0 0 0" rpy="0 0 0"/>
         <geometry>
-          <mesh filename="package://iiwa_description/meshes/iiwa7/visual/link_6.stl"/>
-        </geometry>
-        <material name="Orange"/>
-      </visual>
-      <collision>
-        <origin xyz="0 0 0" rpy="0 0 0"/>
-        <geometry>
-          <mesh filename="package://iiwa_description/meshes/iiwa7/collision/link_6.stl"/>
+          <mesh filename="package://kuka_iiwa_support/meshes/iiwa7/visual/link_6.stl"/>
+        </geometry>
+        <material name="Orange"/>
+      </visual>
+      <collision>
+        <origin xyz="0 0 0" rpy="0 0 0"/>
+        <geometry>
+          <mesh filename="package://kuka_iiwa_support/meshes/iiwa7/collision/link_6.stl"/>
         </geometry>
         <material name="Orange"/>
@@ -249,5 +249,5 @@
         <origin xyz="0 0 -0.0005" rpy="0 0 0"/>
         <geometry>
-          <mesh filename="package://iiwa_description/meshes/iiwa7/visual/link_7.stl"/>
+          <mesh filename="package://kuka_iiwa_support/meshes/iiwa7/visual/link_7.stl"/>
         </geometry>
         <material name="Grey"/>
@@ -256,5 +256,5 @@
         <origin xyz="0 0 -0.0005" rpy="0 0 0"/>
         <geometry>
-          <mesh filename="package://iiwa_description/meshes/iiwa7/collision/link_7.stl"/>
+          <mesh filename="package://kuka_iiwa_support/meshes/iiwa7/collision/link_7.stl"/>
         </geometry>
         <material name="Grey"/>

File: rl_robot_description_pkg/urdf/pan_tilt_generated.urdf (robot description, URDF)
Before this commit: robot pan_tilt, 3 links, 2 joints
Links:
- removed link base_link
- removed link pan_link
- removed link tilt_link
Joints:
- removed joint pan_joint
- removed joint tilt_joint
